File: kicad/mushi-rounded.kicad_pcb (KiCad board)
At the start: 2 copper layers, 261 x 90.8 mm, 86 parts

Commit message: new routing
Routing:
- net rGND: track 520.6 -> 509.5 mm
- net GND: track 501.2 -> 490.7 mm
- net mirror_matrix_ring_bottom: track 111.1 -> 107.5 mm
- net mirror_thumbs_inner_cluster: track 93.8 -> 90.4 mm
- net matrix_pinky_bottom: track 153.3 -> 150.3 mm
- net mirror_thumbs_middle_cluster: track 75.0 -> 72.3 mm
- net mirror_thumbs_outer_cluster: track 64.3 -> 62.2 mm
- net mirror_matrix_pinky_top: track 110.4 -> 108.4 mm
- net mirror_matrix_ring_top: track 87.5 -> 85.6 mm
- net rP3V3: track 39.2 -> 37.3 mm
- net matrix_middle_top: track 87.4 -> 85.6 mm
- net matrix_pinky_top: track 129.3 -> 127.5 mm
- net mirror_matrix_ring_middle: track 88.8 -> 90.6 mm
- net matrix_middle_middle: track 89.4 -> 87.6 mm
- net matrix_ring_bottom: track 123.0 -> 121.3 mm
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