File: kicad/mushi.kicad_pcb (KiCad board)
At the start: 2 copper layers, 261 x 90.8 mm, 86 parts

Commit message: new routing
Routing:
- net rGND: track 520.6 -> 0.00 mm
- net GND: track 501.2 -> 0.00 mm
- net mirror_matrix_pinky_top: track 110.4 -> 126.1 mm
- net mirror_matrix_middle_top: track 70.0 -> 82.9 mm
- net mirror_matrix_pinky_middle: track 112.9 -> 125.2 mm
- net mirror_thumbs_middle_cluster: track 73.6 -> 84.3 mm
- net mirror_thumbs_inner_cluster: track 92.5 -> 102.4 mm
- net mirror_matrix_middle_bottom: track 81.2 -> 91.0 mm
- net mirror_matrix_middle_middle: track 69.7 -> 79.5 mm
- net mirror_matrix_ring_top: track 87.5 -> 96.6 mm
- net mirror_matrix_index_top: track 46.7 -> 54.4 mm
- net mirror_matrix_ring_middle: track 88.8 -> 95.5 mm
- net mirror_matrix_index_middle: track 44.9 -> 50.4 mm
- net mirror_matrix_ring_bottom: track 106.2 -> 111.0 mm
- net mirror_matrix_outer_middle: track 23.3 -> 27.3 mm
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- added copper zone on B.Cu, net GND
- added copper zone on B.Cu, net rGND
